File: Design/H00R7.sch (EAGLE design)
At the start: 1 part, among them P1 HEXABIT_17.32

Commit message: -Remove the modul PN from the silkscreen -Update the logo in the schematic
Other:
- note added: "H00R7"
- note added: "H00R7_Frontend"
- note removed: "0"
- note removed: "H00R70"
- note removed: "H00R70_Frontend"
